File: hardware/rgb-led-v2.kicad_pcb (KiCad board)
At the start: 2 copper layers, 20 x 25 mm, 26 parts, among them P1 CON-SENSOR2, P2 DEBUG, P3 BOOT, U1 XMC1XXX24, U3 DRILL, U4 DRILL, U5 DRILL, U6 DRILL

Commit message: fix schematic version, specify rgb led
Parts:
- D2: value RGB-LED -> QBLP679E-RGB
Changed lines of the file:
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@@
   )
   (layers
-    (0 Vorderseite signal)
-    (31 Rückseite signal)
+    (0 Vorderseite signal hide)
+    (31 Rückseite signal hide)
     (32 B.Adhes user)
     (33 F.Adhes user)
@@
     (aux_axis_origin 176.9 165.9)
     (grid_origin 176.9 165.9)
-    (visible_elements FFFFFFBF)
+    (visible_elements FFFEFFFF)
     (pcbplotparams
-      (layerselection 0x00030_80000001)
+      (layerselection 0x010fc_ffffffff)
       (usegerberextensions true)
       (usegerberattributes false)
@@
       (drillshape 0)
       (scaleselection 1)
-      (outputdirectory "prod/"))
+      (outputdirectory "pcb/"))
   )
   (net 0 "")
@@
     (at 141.9 118.1 270)
     (fp_text reference D2 (at 0.1 0 270) (layer F.Fab)
-      (effects (font (size 0.7 0.7) (thickness 0.15)))
-    )
-    (fp_text value RGB-LED (at 0 3.2 270) (layer F.Fab)
-      (effects (font (size 0.7 0.7) (thickness 0.15)))
+      (effects (font (size 0.35 0.35) (thickness 0.0875)))
+    )
+    (fp_text value QBLP679E-RGB (at -1.4 3.1 270) (layer F.Fab)
+      (effects (font (size 0.35 0.35) (thickness 0.0875)))
     )
     (fp_line (start 2.4 1.6) (end 2.5 1.5) (layer F.Fab) (width 0.3))

Commit message: changed procesor to XMC1100
Parts:
- U1: value XMC1XXX24 -> XMC1100
Changed lines of the file:
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@@
       (effects (font (size 0.3 0.3) (thickness 0.075)))
     )
-    (fp_text value XMC1XXX24 (at 0 0.8) (layer F.Fab)
+    (fp_text value XMC1100 (at 0 0.8) (layer F.Fab)
       (effects (font (size 0.3 0.3) (thickness 0.075)))
     )
